File: schematics/pico_test_synth1.brd (EAGLE design)
At the start: 152.4 x 68.6 mm, 49 parts, among them IC1 H11L1MS, J1 AUDIO-JACK-TRRS, J2 AUDIO-JACK-TRRS, P1 10k, P2 10k, U1 PICO, U2 I2S_PCM_51XX_SOUNDCARD

Commit message: route +5V to PCM5102 module instead of +3V3, fixes #2
Connections:
- removed net N$5: U1.39, U1.P$39
- new net +5V: U1.39, U1.P$39, U2.VIN
- net +3V3: no longer U2.VIN
Routing:
- net +5V: track 0.00 -> 144.3 mm
- net +3V3: track 307.6 -> 184.5 mm
- net SW: track 113.9 -> 117.6 mm
- net TPAD11: track 90.5 -> 94.1 mm
- net POTB: track 122.6 -> 124.4 mm, vias 1 -> 2
- net POTA: track 90.8 -> 92.0 mm, vias 0 -> 1
- net N$5: track 1.11 -> 0.00 mm
- net TPAD12: track 102.2 -> 103.0 mm
- net TPAD13: track 113.0 -> 113.7 mm
Other:
- board text added: "15 Feb 2025 - @todbot"
- board text removed: "6 Aug 2023 - @todbot"
