File: schematics/pico_test_synth1.sch (EAGLE design)
At the start: 49 parts, among them IC1 H11L1MS, J1 AUDIO-JACK-TRRS, J2 AUDIO-JACK-TRRS, P1 10k, P2 10k, U1 PICO, U2 I2S_PCM_51XX_SOUNDCARD

Commit message: route +5V to PCM5102 module instead of +3V3, fixes #2
Connections:
- removed net N$5: U1.VSYS
- new net +5V: U1.VSYS, U2.VIN
- net +3V3: no longer U2.VIN
Changed lines of the file:
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@@
 <part name="GND26" library="supply1" library_urn="urn:adsk.eagle:library:371" deviceset="GND" device=""/>
 <part name="GND27" library="supply1" library_urn="urn:adsk.eagle:library:371" deviceset="GND" device=""/>
-<part name="+3V3" library="supply1" library_urn="urn:adsk.eagle:library:371" deviceset="+3V3" device=""/>
 <part name="GND28" library="supply1" library_urn="urn:adsk.eagle:library:371" deviceset="GND" device=""/>
 <part name="R18" library="rcl" library_urn="urn:adsk.eagle:library:334" deviceset="R-EU_" device="R0805" package3d_urn="urn:adsk.eagle:package:23553/2" value="33"/>
@@
 <part name="+3V4" library="supply1" library_urn="urn:adsk.eagle:library:371" deviceset="+3V3" device=""/>
 <part name="GND2" library="supply1" library_urn="urn:adsk.eagle:library:371" deviceset="GND" device=""/>
+<part name="P+1" library="supply1" library_urn="urn:adsk.eagle:library:371" deviceset="+5V" device=""/>
+<part name="P+2" library="supply1" library_urn="urn:adsk.eagle:library:371" deviceset="+5V" device=""/>
 </parts>
 <sheets>
@@
 <attribute name="VALUE" x="162.56" y="88.9" size="1.778" layer="96" rot="R270"/>
 </instance>
-<instance part="+3V3" gate="G$1" x="157.48" y="83.82" smashed="yes" rot="MR270">
-<attribute name="VALUE" x="157.226" y="82.042" size="1.778" layer="96" rot="MR0"/>
-</instance>
 <instance part="GND28" gate="1" x="165.1" y="96.52" smashed="yes" rot="R270">
 <attribute name="VALUE" x="162.56" y="99.06" size="1.778" layer="96" rot="R270"/>
@@
 <instance part="GND2" gate="1" x="63.5" y="124.46" smashed="yes" rot="MR0">
 <attribute name="VALUE" x="66.04" y="121.92" size="1.778" layer="96" rot="MR0"/>
+</instance>
+<instance part="P+1" gate="1" x="76.2" y="195.58" smashed="yes" rot="R270">
+<attribute name="VALUE" x="78.74" y="195.58" size="1.778" layer="96"/>
+</instance>
+<instance part="P+2" gate="1" x="157.48" y="83.82" smashed="yes" rot="R90">
+<attribute name="VALUE" x="154.94" y="83.82" size="1.778" layer="96" rot="R180"/>
 </instance>
 </instances>
@@
 </segment>
 <segment>
-<pinref part="U2" gate="G$1" pin="VIN"/>
-<pinref part="+3V3" gate="G$1" pin="+3V3"/>
-<wire x1="160.02" y1="83.82" x2="187.96" y2="83.82" width="0.1524" layer="91"/>
-</segment>
-<segment>
 <pinref part="R18" gate="G$1" pin="1"/>
 <wire x1="177.8" y1="142.24" x2="162.56" y2="142.24" width="0.1524" layer="91"/>
@@
 </segment>
 </net>
-<net name="N$5" class="0">
+<net name="N$6" class="0">
+<segment>
+<pinref part="U1" gate="G$1" pin="VBUS"/>
+<wire x1="63.5" y1="198.12" x2="68.58" y2="198.12" width="0.1524" layer="91"/>
+</segment>
+</net>
+<net name="+5V" class="0">
 <segment>
 <pinref part="U1" gate="G$1" pin="VSYS"/>
 <wire x1="63.5" y1="195.58" x2="68.58" y2="195.58" width="0.1524" layer="91"/>
-</segment>
-</net>
-<net name="N$6" class="0">
-<segment>
-<pinref part="U1" gate="G$1" pin="VBUS"/>
-<wire x1="63.5" y1="198.12" x2="68.58" y2="198.12" width="0.1524" layer="91"/>
-</segment>
-</net>
+<pinref part="P+1" gate="1" pin="+5V"/>
+<wire x1="73.66" y1="195.58" x2="68.58" y2="195.58" width="0.1524" layer="91"/>
+</segment>
+<segment>
+<pinref part="U2" gate="G$1" pin="VIN"/>
+<wire x1="160.02" y1="83.82" x2="187.96" y2="83.82" width="0.1524" layer="91"/>
+<pinref part="P+2" gate="1" pin="+5V"/>
+</segment>
+</net>
