File: schematics/pico_test_synth2/pico_test_synth2.kicad_pcb (KiCad board)
At the start: 2 copper layers, 152.4 x 68.6 mm, 55 parts, among them IC1 H11L1, J1 AudioJack4, J2 AudioJack4, SW1 SW_Push, U1 Pico

Commit message: fixes
Parts:
- moved POT2 0.54 mm to (148.2, 42.1)
- moved POT1 0.45 mm to (117.7, 42.1)
Routing:
- net /I2S_BCK: track 109.3 -> 109.8 mm
Other:
- board text added: "- +"
- board text added: "PCM5102 module"
- board text added: "TRS-A"
- board text added: "Vin Gnd I2S LRCK I2S DATA I2S BCK"

Commit message: fixes
Other:
- board text added: "﻿Parts: - Raspberry Pi Pico (Pico2 if touchpad pull jumper changed) - 0.9{dblquote} I2C OLED SSD1306 display - PCM5102 I2S DAC module - 2x 10k pots, 9mm - tact switch 6mm - 2x PJ320D 3.5mm jacks - IC1: H11L1 optoisolator - D1: 1N4148 - R1-R16: 1M, R7: 10, R18: 33 R19,R21,R22: 4.7k, R20: 220 - C1:00nF"
- board text removed: "﻿Parts: - Raspberry Pi Pico - 0.9{dblquote} I2C OLED SSD1306 display - PCM5102 I2S DAC module - 2x 10k pots, 9mm - tact switch 6mm - 2x PJ320D 3.5mm jacks - IC1: H11L1 optoisolator - D1: 1N4148 - R1-R16: 1M, R7: 10, R18: 33 R19,R21,R22: 4.7k, R20: 220 - C1:00nF"
Changed lines of the file:
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@@
 		)
 		(group ""
-			(members "1010ae21-8e28-434d-86e3-995909ba90c2")
+			(members "136127d9-39d5-4bd6-9dd0-fdb8b51620e7")
 		)
 		(embedded_fonts no)
@@
 		)
 	)
-	(gr_text "﻿Parts:\n- Raspberry Pi Pico \n- 0.9{dblquote} I2C OLED SSD1306 display\n- PCM5102 I2S DAC module\n- 2x 10k pots, 9mm\n- tact switch 6mm\n- 2x PJ320D 3.5mm jacks\n- IC1: H11L1 optoisolator\n- D1: 1N4148\n- R1-R16: 1M, R7: 10, R18: 33 R19,R21,R22: 4.7k, R20: 220\n- C1:00nF"
+	(gr_text "﻿Parts:\n- Raspberry Pi Pico (Pico2 if touchpad pull jumper changed)\n- 0.9{dblquote} I2C OLED SSD1306 display\n- PCM5102 I2S DAC module\n- 2x 10k pots, 9mm\n- tact switch 6mm\n- 2x PJ320D 3.5mm jacks\n- IC1: H11L1 optoisolator\n- D1: 1N4148\n- R1-R16: 1M, R7: 10, R18: 33 R19,R21,R22: 4.7k, R20: 220\n- C1:00nF"
 		(at 106.3 80.043 0)
 		(layer "B.SilkS")

Commit message: fixes
Routing:
- net +3V3: track 197.1 -> 194.1 mm
- net /SW: track 112.6 -> 113.7 mm
- net GND: vias 0 -> 11
Other:
- board text added: "danger: only connect one! touchpad pull gnd 3v3"
- board text removed: "gnd 3v3 touchpad pull"

Commit message: pcb2 cleanup before production
Changed lines of the file:
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@@
+	)
+	(segment
+		(start 150.67 47.324)
+		(end 150.67 48.801)
+		(width 0.3048)
+		(layer "F.Cu")
+		(net 1)
 	)
 	(segment
@@
 	)
 	(segment
-		(start 118.238 30.64)
-		(end 118.238 31.402)
-		(width 0.3048)
-		(layer "F.Cu")
-		(net 1)
-	)
-	(segment
-		(start 150.67 47.324)
-		(end 148.21 44.864)
-		(width 0.3048)
-		(layer "F.Cu")
-		(net 1)
-	)
-	(segment
 		(start 105.538 34.717)
 		(end 105.538 35.707)
@@
 	)
 	(segment
-		(start 125.858 44.864)
-		(end 125.858 39.022)
-		(width 0.3048)
-		(layer "F.Cu")
-		(net 1)
-	)
-	(segment
 		(start 105.017 34.196)
 		(end 105.538 34.717)
@@
 	)
 	(segment
+		(start 126.112 39.276)
+		(end 126.112 44.864)
+		(width 0.3048)
+		(layer "F.Cu")
+		(net 1)
+	)
+	(segment
 		(start 96.648 42.832)
 		(end 94.870001 44.609999)
@@
 	)
 	(segment
-		(start 118.746 30.132)
-		(end 118.238 30.64)
+		(start 126.112 60.104)
+		(end 126.112 44.864)
 		(width 0.3048)
 		(layer "F.Cu")
@@
 	)
 	(segment
-		(start 123.445 48.801)
-		(end 123.445 47.277)
-		(width 0.3048)
-		(layer "F.Cu")
-		(net 1)
-	)
-	(segment
 		(start 100.204 33.18)
 		(end 101.22 34.196)
@@
 	)
 	(segment
-		(start 119.445 30.132)
-		(end 118.746 30.132)
-		(width 0.3048)
-		(layer "F.Cu")
-		(net 1)
-	)
-	(segment
-		(start 125.858 39.022)
-		(end 118.238 31.402)
-		(width 0.3048)
-		(layer "F.Cu")
-		(net 1)
-	)
-	(segment
 		(start 101.22 34.196)
 		(end 105.017 34.196)
@@
 	)
 	(segment
-		(start 150.67 48.801)
-		(end 150.67 47.324)
-		(width 0.3048)
-		(layer "F.Cu")
-		(net 1)
-	)
-	(segment
-		(start 126.112 60.104)
-		(end 126.112 51.468)
+		(start 119.381 32.545)
+		(end 119.445 32.481)
 		(width 0.3048)
 		(layer "F.Cu")
@@
 	)
 	(segment
-		(start 126.112 51.468)
-		(end 123.445 48.801)
-		(width 0.3048)
-		(layer "F.Cu")
-		(net 1)
-	)
-	(segment
-		(start 148.21 44.864)
-		(end 125.858 44.864)
-		(width 0.3048)
-		(layer "F.Cu")
-		(net 1)
-	)
-	(segment
 		(start 76.963 30.195)
 		(end 76.963 31.275)
@@
 	)
 	(segment
+		(start 120.19 48.801)
+		(end 126.112 48.801)
+		(width 0.3048)
+		(layer "F.Cu")
+		(net 1)
+	)
+	(segment
 		(start 105.601 39.276)
 		(end 105.538 39.339)
@@
 	)
 	(segment
-		(start 120.19 48.801)
-		(end 123.445 48.801)
-		(width 0.3048)
-		(layer "F.Cu")
-		(net 1)
-	)
-	(segment
 		(start 103.252 42.832)
 		(end 96.648 42.832)
@@
 	)
 	(segment
+		(start 126.112 44.864)
+		(end 148.21 44.864)
+		(width 0.3048)
+		(layer "F.Cu")
+		(net 1)
+	)
+	(segment
 		(start 105.551 35.72)
 		(end 105.551 39.226)
@@
 	)
 	(segment
+		(start 148.21 44.864)
+		(end 150.67 47.324)
+		(width 0.3048)
+		(layer "F.Cu")
+		(net 1)
+	)
+	(segment
 		(start 105.538 40.546)
 		(end 103.252 42.832)
@@
 	)
 	(segment
-		(start 123.445 47.277)
-		(end 125.858 44.864)
+		(start 119.381 32.545)
+		(end 126.112 39.276)
+		(width 0.3048)
+		(layer "F.Cu")
+		(net 1)
+	)
+	(segment
+		(start 119.445 32.481)
+		(end 119.445 30.132)
 		(width 0.3048)
 		(layer "F.Cu")
@@
 	)
 	(via
-		(at 118.238 31.402)
+		(at 119.381 32.545)
 		(size 0.6)
 		(drill 0.3)
@@
 		(drill 0.3)
 		(layers "F.Cu" "B.Cu")
-		(net 1)
-	)
-	(segment
-		(start 116.46 33.18)
-		(end 118.238 31.402)
-		(width 0.3048)
-		(layer "B.Cu")
 		(net 1)
 	)
@@
 	)
 	(segment
+		(start 119.381 32.545)
+		(end 118.746 33.18)
+		(width 0.3048)
+		(layer "B.Cu")
+		(net 1)
+	)
+	(segment
 		(start 30.16 26.636)
 		(end 32.259 28.735)
@@
 	)
 	(segment
+		(start 118.746 33.18)
+		(end 100.204 33.18)
+		(width 0.3048)
+		(layer "B.Cu")
+		(net 1)
+	)
+	(segment
 		(start 126.366 60.104)
 		(end 126.395999 60.133999)
@@
 		(width 0.3048)
 		(layer "B.Cu")
-		(net 1)
-	)
-	(segment
-		(start 100.204 33.18)
-		(end 116.46 33.18)
-		(width 0.3048)
-		(layer "B.Cu")

Commit message: pico_test_synth2 updates
Parts:
- TP1, TP10, TP11, TP12, TP13, TP14, TP15, TP16, TP2, TP3, TP4, TP5, TP6, TP7, TP8, TP9: footprint todbot_stuff:Pad-CapTouch-10mm-roundrect -> todbot_stuff:Pad-CapTouch-11_2mm-roundrect
Other:
- board text added: "github.com/todbot/pico_test_synth works with CircuitPython! 4 May 2025 pico_test_synth2"
- board text removed: "github.com/todbot/pico_test_synth works with CircuitPython! 15 Apr 2025 pico_test_synth2"

Commit message: pico_test_synth2 5Jun2025 production run
Parts:
- removed JP3: Jumper_2_Open, Jumper:SolderJumper-2_P1.3mm_Open_RoundedPad1.0x1.5mm
- added JP1: SolderJumper_2_Bridged, Jumper:SolderJumper-2_P1.3mm_Bridged_RoundedPad1.0x1.5mm, B.Cu at (128.1, 59.5)
- JP2: value Jumper_2_Bridged -> SolderJumper_2_Open; footprint Jumper:SolderJumper-2_P1.3mm_Bridged_RoundedPad1.0x1.5mm -> Jumper:SolderJumper-2_P1.3mm_Open_RoundedPad1.0x1.5mm
- R19: value 4k7 -> 4.7k
Other:
- board text added: "Raspberry Pi Pico2 (or Pico)"
- board text added: "Raspberry Pi Pico2 / Pico"
- board text added: "github.com/todbot/pico_test_synth works with CircuitPython! 5 Jun 2025 pico_test_synth2"
- board text added: "pico_test_synth2"
- board text added: "﻿Parts: - Raspberry Pi Pico2 (or Pico) - 0.9{dblquote} I2C OLED SSD1306 display - PCM5102 I2S DAC module - 2x 10k pots, 9mm - tact switch 6mm - 2x PJ320D 3.5mm jacks - IC1: H11L1 optoisolator - D1: 1N4148 - R1-R16: 1M, R7: 10, R18: 33 R19,R21,R22: 4.7k, R20: 220 - C1:00nF"
- board text removed: "github.com/todbot/pico_test_synth works with CircuitPython! 4 May 2025 pico_test_synth2"
- board text removed: "pico_test_synth"
- board text removed: "raspberry pi pico"
- board text removed: "﻿Parts: - Raspberry Pi Pico (Pico2 if touchpad pull jumper changed) - 0.9{dblquote} I2C OLED SSD1306 display - PCM5102 I2S DAC module - 2x 10k pots, 9mm - tact switch 6mm - 2x PJ320D 3.5mm jacks - IC1: H11L1 optoisolator - D1: 1N4148 - R1-R16: 1M, R7: 10, R18: 33 R19,R21,R22: 4.7k, R20: 220 - C1:00nF"
Changed lines of the file:
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@@
 			(at -0.1 2.9 180)
 			(layer "B.Fab")
+			(hide yes)
 			(effects
 				(font
@@
 			)
 		)
-		(property "Value" "4k7"
+		(property "Value" "4.7k"
 			(at 0 1.43 0)
 			(layer "F.Fab")
@@
 		)
 	)
-	(footprint "Jumper:SolderJumper-2_P1.3mm_Open_RoundedPad1.0x1.5mm"
+	(footprint "Jumper:SolderJumper-2_P1.3mm_Bridged_RoundedPad1.0x1.5mm"
 		(layer "B.Cu")
-		(at 128.144 59.484 90)
-		(descr "SMD Solder Jumper, 1x1.5mm, rounded Pads, 0.3mm gap, open")
-		(tags "solder jumper open")
-		(property "Reference" "JP3"
-			(at -2.398 0 0)
+		(at 128.144 59.483999 90)
+		(descr "SMD Solder Jumper, 1x1.5mm, rounded Pads, 0.3mm gap, bridged with 1 copper strip")
+		(tags "net tie solder jumper bridged")
+		(property "Reference" "JP1"
+			(at -2.398001 0 0)
 			(layer "B.SilkS")
 			(effects
@@
 			)
 		)
-		(property "Value" "Jumper_2_Open"
+		(property "Value" "SolderJumper_2_Bridged"
 			(at 0 -1.9 90)
 			(layer "B.Fab")
@@
 			)
 		)
-		(property "Description" "Jumper, 2-pole, open"
+		(property "Description" "Solder Jumper, 2-pole, closed/bridged"
 			(at 0 0 270)
 			(unlocked yes)
@@
 			)
 		)
-		(property ki_fp_filters "Jumper* TestPoint*2Pads* TestPoint*Bridge*")
+		(property ki_fp_filters "SolderJumper*Bridged*")
 		(sheetname "/")
 		(sheetfile "pico_test_synth2.kicad_sch")
 		(zone_connect 1)
-		(attr exclude_from_pos_files allow_soldermask_bridges)
+		(attr exclude_from_pos_files exclude_from_bom allow_soldermask_bridges)
+		(net_tie_pad_groups "1, 2")
+		(fp_poly
+			(pts
+				(xy 0.25 0.3) (xy -0.25 0.3) (xy -0.25 -0.3) (xy 0.25 -0.3)
+			)
+			(stroke
+				(width 0)
+				(type solid)
+			)
+			(fill yes)
+			(layer "B.Cu")
+		)
 		(fp_poly
 			(pts
@@
 		(embedded_fonts no)
 	)
-	(footprint "Jumper:SolderJumper-2_P1.3mm_Bridged_RoundedPad1.0x1.5mm"
+	(footprint "Jumper:SolderJumper-2_P1.3mm_Open_RoundedPad1.0x1.5mm"
 		(layer "B.Cu")
 		(at 133.478 59.484 90)
-		(descr "SMD Solder Jumper, 1x1.5mm, rounded Pads, 0.3mm gap, bridged with 1 copper strip")
-		(tags "net tie solder jumper bridged")
+		(descr "SMD Solder Jumper, 1x1.5mm, rounded Pads, 0.3mm gap, open")
+		(tags "solder jumper open")
 		(property "Reference" "JP2"
-			(at -2.398 0 0)
+			(at -2.398 0 180)
 			(layer "B.SilkS")
 			(effects
@@
 			)
 		)
-		(property "Value" "Jumper_2_Bridged"
-			(at 0 -1.9 90)
+		(property "Value" "SolderJumper_2_Open"
+			(at 0 -1.9 270)
 			(layer "B.Fab")
 			(hide yes)
@@
 			)
 		)
-		(property "Description" "Jumper, 2-pole, closed/bridged"
+		(property "Description" "Solder Jumper, 2-pole, open"
 			(at 0 0 270)
 			(unlocked yes)
@@
 			)
 		)
-		(property ki_fp_filters "Jumper* TestPoint*2Pads* TestPoint*Bridge*")
+		(property ki_fp_filters "SolderJumper*Open*")
 		(sheetname "/")
 		(sheetfile "pico_test_synth2.kicad_sch")
 		(zone_connect 1)
-		(attr exclude_from_pos_files allow_soldermask_bridges)
-		(net_tie_pad_groups "1, 2")
-		(fp_poly
-			(pts
-				(xy 0.25 0.3) (xy -0.25 0.3) (xy -0.25 -0.3) (xy 0.25 -0.3)
-			)
-			(stroke
-				(width 0)
-				(type solid)
-			)
-			(fill yes)
-			(layer "B.Cu")
-		)
-		(fp_poly
-			(pts
-				(xy -0.15 0.75) (xy 0.15 0.75) (xy 0.15 -0.75) (xy -0.15 -0.75)
-			)
+		(attr exclude_from_pos_files exclude_from_bom allow_soldermask_bridges)
+		(fp_rect
+			(start -0.15 0.75)
+			(end 0.15 -0.75)
 			(stroke
 				(width 0)
@@
 		)
 		(fp_line
-			(start -1.4 -0.300001)
-			(end -1.4 0.300001)
+			(start -1.4 -0.3)
+			(end -1.4 0.3)
 			(stroke
 				(width 0.12)
@@
 		)
 		(fp_line
-			(start 1.4 0.300001)
-			(end 1.4 -0.300001)
+			(start 1.4 0.3)
+			(end 1.4 -0.3)
 			(stroke
 				(width 0.12)
@@
 		(fp_arc
 			(start 0.7 -1)
-			(mid 1.194974 -0.794975)
-			(end 1.4 -0.300001)
+			(mid 1.194975 -0.794975)
+			(end 1.4 -0.3)
 			(stroke
 				(width 0.12)
@@
 		)
 		(fp_arc
-			(start -1.4 -0.300001)
+			(start -1.4 -0.3)
 			(mid -1.194975 -0.794975)
 			(end -0.7 -1)
@@
 		)
 		(fp_arc
-			(start 1.4 0.300001)
-			(mid 1.194974 0.794975)
+			(start 1.4 0.3)
+			(mid 1.194975 0.794975)
 			(end 0.7 1)
 			(stroke
@@
 			(start -0.7 1)
 			(mid -1.194975 0.794975)
-			(end -1.4 0.300001)
+			(end -1.4 0.3)
 			(stroke
 				(width 0.12)
@@
 		)
 		(pad "1" smd custom
-			(at -0.649999 0 90)
+			(at -0.65 0 90)
 			(size 1 0.5)
 			(layers "B.Cu" "B.Mask")
@@
 		)
 		(pad "2" smd custom
-			(at 0.649999 0 90)
+			(at 0.65 0 90)
 			(size 1 0.5)
 			(layers "B.Cu" "B.Mask")
@@
 		)
 	)
-	(gr_text "pico_test_synth"
+	(gr_text "pico_test_synth2"
 		(at 167.26 52.23 90)
 		(layer "F.SilkS")
@@
 		)
 	)
-	(gr_text "raspberry pi pico"
-		(at 44.13 33.09 0)
+	(gr_text "Raspberry Pi Pico2 / Pico"
+		(at 24.766 33.18 0)
 		(layer "F.SilkS")
 		(effects
@@
 		)
 	)
+	(gr_text "Raspberry Pi Pico2 (or Pico)"
+		(at 39.752 33.18 0)
+		(layer "B.SilkS")
+		(effects
+			(font
+				(size 1.524 1.397)
+				(thickness 0.3048)
+				(bold yes)
+			)
+			(justify mirror)
+		)
+	)
 	(gr_text "PCM5102 module"
 		(at 141.86 24.544 0)
@@
 		)
 	)
-	(gr_text "pico_test_synth"
+	(gr_text "pico_test_synth2"
 		(at 161.291 67.851 0)
 		(layer "B.SilkS")
@@
 		)
 	)
-	(gr_text "github.com/todbot/pico_test_synth\nworks with CircuitPython!\n4 May 2025\n\npico_test_synth2"
+	(gr_text "github.com/todbot/pico_test_synth\nworks with CircuitPython!\n5 Jun 2025\n\npico_test_synth2"
 		(at 161.291 80.043 0)
 		(layer "B.SilkS")
@@
 		)
 	)
-	(gr_text "﻿Parts:\n- Raspberry Pi Pico (Pico2 if touchpad pull jumper changed)\n- 0.9{dblquote} I2C OLED SSD1306 display\n- PCM5102 I2S DAC module\n- 2x 10k pots, 9mm\n- tact switch 6mm\n- 2x PJ320D 3.5mm jacks\n- IC1: H11L1 optoisolator\n- D1: 1N4148\n- R1-R16: 1M, R7: 10, R18: 33 R19,R21,R22: 4.7k, R20: 220\n- C1:00nF"
+	(gr_text "﻿Parts:\n- Raspberry Pi Pico2 (or Pico)\n- 0.9{dblquote} I2C OLED SSD1306 display\n- PCM5102 I2S DAC module\n- 2x 10k pots, 9mm\n- tact switch 6mm\n- 2x PJ320D 3.5mm jacks\n- IC1: H11L1 optoisolator\n- D1: 1N4148\n- R1-R16: 1M, R7: 10, R18: 33 R19,R21,R22: 4.7k, R20: 220\n- C1:00nF"
 		(at 106.3 80.043 0)
 		(layer "B.SilkS")
@@
 	)
 	(segment
-		(start 116.841 46.261)
-		(end 117.727411 47.147411)
+		(start 71.779049 41.331049)
+		(end 104.037049 41.331049)
 		(width 0.25)
 		(layer "B.Cu")
@@
 	)
 	(segment
-		(start 103.633 40.927)
-		(end 108.967 46.261)
+		(start 70.232 39.784)
+		(end 71.779049 41.331049)
 		(width 0.25)
 		(layer "B.Cu")
@@
 	)
 	(segment
-		(start 71.375 40.927)
-		(end 103.633 40.927)
+		(start 104.037049 41.331049)
+		(end 108.967 46.261)
 		(width 0.25)
 		(layer "B.Cu")
@@
 	)
 	(segment
-		(start 70.232 39.784)
-		(end 71.375 40.927)
+		(start 108.967 46.261)
+		(end 116.841 46.261)
 		(width 0.25)
 		(layer "B.Cu")
@@
 	)
 	(segment
-		(start 108.967 46.261)
-		(end 116.841 46.261)
+		(start 42.86 32.037)
+		(end 42.86 35.526)
 		(width 0.25)
 		(layer "B.Cu")
@@
 	)
 	(segment
-		(start 42.86 32.037)
-		(end 42.86 35.526)
+		(start 42.86 35.526)
+		(end 47.118 39.784)
 		(width 0.25)
 		(layer "B.Cu")
@@
 	)
 	(segment
-		(start 42.86 35.526)
-		(end 47.118 39.784)
+		(start 116.841 46.261)
+		(end 117.727411 47.147411)
 		(width 0.25)
 		(layer "B.Cu")
