File: schematics/pico_test_synth2/pico_test_synth2.kicad_sch (KiCad schematic)
At the start: 55 parts, among them IC1 H11L1, J1 AudioJack4, J2 AudioJack4, SW1 SW_Push, U1 Pico

Commit message: pcb2 cleanup before production
Parts:
- POT1, POT2: footprint PCM_4ms_Potentiometer:Pot_9mm_DShaft -> 4ms_Potentiometer:Pot_9mm_DShaft
Connections:
- no-connect marks 14 -> 13
Other:
- note added: "touchpull jumpers - defaults to pull to GND, for Pico RP2040 - can switch to pull to 3V3, for Pico2 RP2350 - DANGER: only set ONE jumper"
- moved on the sheet: C1, D1, H1, H2, H3, H4, IC1, J1, J2, POT1A, POT2A, R17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

Commit message: pico_test_synth2 updates
Parts:
- TP1, TP10, TP11, TP12, TP13, TP14, TP15, TP16, TP2, TP3, TP4, TP5, TP6, TP7, TP8, TP9: footprint todbot_stuff:Pad-CapTouch-10mm-roundrect -> todbot_stuff:Pad-CapTouch-11_2mm-roundrect
Changed lines of the file:
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@@
 			)
 		)
-		(property "Footprint" "todbot_stuff:Pad-CapTouch-10mm-roundrect"
+		(property "Footprint" "todbot_stuff:Pad-CapTouch-11_2mm-roundrect"
 			(at 203.2 146.05 0)
 			(effects
@@
 			)
 		)
-		(property "Footprint" "todbot_stuff:Pad-CapTouch-10mm-roundrect"
+		(property "Footprint" "todbot_stuff:Pad-CapTouch-11_2mm-roundrect"
 			(at 248.92 146.05 0)
 			(effects
@@
 			)
 		)
-		(property "Footprint" "todbot_stuff:Pad-CapTouch-10mm-roundrect"
+		(property "Footprint" "todbot_stuff:Pad-CapTouch-11_2mm-roundrect"
 			(at 261.62 113.03 0)
 			(effects
@@
 			)
 		)
-		(property "Footprint" "todbot_stuff:Pad-CapTouch-10mm-roundrect"
+		(property "Footprint" "todbot_stuff:Pad-CapTouch-11_2mm-roundrect"
 			(at 191.77 146.05 0)
 			(effects
@@
 			)
 		)
-		(property "Footprint" "todbot_stuff:Pad-CapTouch-10mm-roundrect"
+		(property "Footprint" "todbot_stuff:Pad-CapTouch-11_2mm-roundrect"
 			(at 193.04 113.03 0)
 			(effects
@@
 			)
 		)
-		(property "Footprint" "todbot_stuff:Pad-CapTouch-10mm-roundrect"
+		(property "Footprint" "todbot_stuff:Pad-CapTouch-11_2mm-roundrect"
 			(at 238.76 113.03 0)
 			(effects
@@
 			)
 		)
-		(property "Footprint" "todbot_stuff:Pad-CapTouch-10mm-roundrect"
+		(property "Footprint" "todbot_stuff:Pad-CapTouch-11_2mm-roundrect"
 			(at 271.78 146.05 0)
 			(effects
@@
 			)
 		)
-		(property "Footprint" "todbot_stuff:Pad-CapTouch-10mm-roundrect"
+		(property "Footprint" "todbot_stuff:Pad-CapTouch-11_2mm-roundrect"
 			(at 260.35 146.05 0)
 			(effects
@@
 			)
 		)
-		(property "Footprint" "todbot_stuff:Pad-CapTouch-10mm-roundrect"
+		(property "Footprint" "todbot_stuff:Pad-CapTouch-11_2mm-roundrect"
 			(at 226.06 146.05 0)
 			(effects
@@
 			)
 		)
-		(property "Footprint" "todbot_stuff:Pad-CapTouch-10mm-roundrect"
+		(property "Footprint" "todbot_stuff:Pad-CapTouch-11_2mm-roundrect"
 			(at 273.05 113.03 0)
 			(effects
@@
 			)
 		)
-		(property "Footprint" "todbot_stuff:Pad-CapTouch-10mm-roundrect"
+		(property "Footprint" "todbot_stuff:Pad-CapTouch-11_2mm-roundrect"
 			(at 214.63 146.05 0)
 			(effects
@@
 			)
 		)
-		(property "Footprint" "todbot_stuff:Pad-CapTouch-10mm-roundrect"
+		(property "Footprint" "todbot_stuff:Pad-CapTouch-11_2mm-roundrect"
 			(at 237.49 146.05 0)
 			(effects
@@
 			)
 		)
-		(property "Footprint" "todbot_stuff:Pad-CapTouch-10mm-roundrect"
+		(property "Footprint" "todbot_stuff:Pad-CapTouch-11_2mm-roundrect"
 			(at 215.9 113.03 0)
 			(effects
@@
 					(size 1.27 1.27)
 				)
-				(hide yes)
 			)
 		)
@@
 			)
 		)
-		(property "Footprint" "todbot_stuff:Pad-CapTouch-10mm-roundrect"
+		(property "Footprint" "todbot_stuff:Pad-CapTouch-11_2mm-roundrect"
 			(at 204.47 113.03 0)
 			(effects
@@
 			)
 		)
-		(property "Footprint" "todbot_stuff:Pad-CapTouch-10mm-roundrect"
+		(property "Footprint" "todbot_stuff:Pad-CapTouch-11_2mm-roundrect"
 			(at 227.33 113.03 0)
 			(effects
@@
 			)
 		)
-		(property "Footprint" "todbot_stuff:Pad-CapTouch-10mm-roundrect"
+		(property "Footprint" "todbot_stuff:Pad-CapTouch-11_2mm-roundrect"
 			(at 250.19 113.03 0)
 			(effects

Commit message: add pico_test_synth2 to readme
Other:
- company: (none) -> todbot
- title: (none) -> pico_test_synth2
Changed lines of the file:
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@@
 	(generator_version "9.0")
 	(paper "A4")
+	(title_block
+		(title "pico_test_synth2")
+		(date "2025-05-15")
+		(company "todbot")
+	)
 	(text "touchpull jumpers\n- defaults to pull to GND, for Pico RP2040\n- can switch to pull to 3V3, for Pico2 RP2350\n- DANGER: only set ONE jumper"
 		(exclude_from_sim no)

Commit message: pico_test_synth2 5Jun2025 production run
Parts:
- removed JP2: Jumper_2_Bridged, Jumper:SolderJumper-2_P1.3mm_Bridged_RoundedPad1.0x1.5mm, symbol Jumper:Jumper_2_Bridged
- removed JP3: Jumper_2_Open, Jumper:SolderJumper-2_P1.3mm_Open_RoundedPad1.0x1.5mm, symbol Jumper:Jumper_2_Open
- added JP1: SolderJumper_2_Bridged, Jumper:SolderJumper-2_P1.3mm_Bridged_RoundedPad1.0x1.5mm, symbol Jumper:SolderJumper_2_Bridged
- added JP2: SolderJumper_2_Open, Jumper:SolderJumper-2_P1.3mm_Open_RoundedPad1.0x1.5mm, symbol Jumper:SolderJumper_2_Open
- R19: value 4k7 -> 4.7k
Connections:
- net +3V3: now also JP1.1 (A)
- net GND: now also JP2.1 (A)
- net TOUCHCOM: now also JP1.2 (B), JP2.2 (B)
Changed lines of the file:
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@@
 	(wire
 		(pts
-			(xy 154.94 119.38) (xy 157.48 119.38)
+			(xy 152.4 119.38) (xy 157.48 119.38)
 		)
 		(stroke
@@
 	(wire
 		(pts
-			(xy 156.21 127) (xy 157.48 127)
+			(xy 153.67 127) (xy 157.48 127)
 		)
 		(stroke
@@
 	(wire
 		(pts
+			(xy 165.1 127) (xy 167.64 127)
+		)
+		(stroke
+			(width 0)
+			(type default)
+		)
+	)
+	(wire
+		(pts
 			(xy 203.2 156.21) (xy 191.77 156.21)
 		)
@@
 	(wire
 		(pts
+			(xy 165.1 119.38) (xy 167.64 119.38)
+		)
+		(stroke
+			(width 0)
+			(type default)
+		)
+	)
+	(wire
+		(pts
 			(xy 193.04 114.3) (xy 193.04 123.19)
 		)
@@
 			)
 		)
-		(property "Value" "4k7"
+		(property "Value" "4.7k"
 			(at 115.57 129.54 90)
 			(effects
@@
 	(symbol
 		(lib_id "power:GND")
-		(at 156.21 127 0)
+		(at 153.67 127 0)
 		(unit 1)
 		(exclude_from_sim no)
@@
 		(dnp no)
 		(property "Reference" "#PWR031"
-			(at 156.21 133.35 0)
+			(at 153.67 133.35 0)
 			(effects
 				(font
@@
 		)
 		(property "Value" "GND"
-			(at 154.686 129.286 0)
+			(at 152.146 129.286 0)
 			(effects
 				(font
@@
 		)
 		(property "Footprint" ""
-			(at 156.21 127 0)
+			(at 153.67 127 0)
 			(effects
 				(font
@@
 		)
 		(property "Datasheet" ""
-			(at 156.21 127 0)
+			(at 153.67 127 0)
 			(effects
 				(font
@@
 		)
 		(property "Description" "Power symbol creates a global label with name \"GND\" , ground"
-			(at 156.21 127 0)
+			(at 153.67 127 0)
 			(effects
 				(font
@@
 	)
 	(symbol
-		(lib_id "Jumper:Jumper_2_Open")
-		(at 162.56 119.38 0)
-		(unit 1)
-		(exclude_from_sim no)
-		(in_bom yes)
-		(on_board yes)
-		(dnp no)
-		(property "Reference" "JP3"
-			(at 162.56 113.03 0)
-			(effects
-				(font
-					(size 1.27 1.27)
-				)
-			)
-		)
-		(property "Value" "Jumper_2_Open"
-			(at 168.402 115.57 0)
-			(effects
-				(font
-					(size 1.27 1.27)
-				)
-			)
-		)
-		(property "Footprint" "Jumper:SolderJumper-2_P1.3mm_Open_RoundedPad1.0x1.5mm"
-			(at 162.56 119.38 0)
-			(effects
-				(font
-					(size 1.27 1.27)
-				)
-				(hide yes)
-			)
-		)
-		(property "Datasheet" "~"
-			(at 162.56 119.38 0)
-			(effects
-				(font
-					(size 1.27 1.27)
-				)
-				(hide yes)
-			)
-		)
-		(property "Description" "Jumper, 2-pole, open"
-			(at 162.56 119.38 0)
-			(effects
-				(font
-					(size 1.27 1.27)
-				)
-				(hide yes)
-			)
-		)
-		(pin "1"
-		)
-		(pin "2"
-		)
-		(instances
-			(project ""
-				(path "/91d40f58-a363-48c7-98aa-eb2459062304"
-					(reference "JP3")
-					(unit 1)
-				)
-			)
-		)
-	)
-	(symbol
 		(lib_id "todbot_stuff:Capacitive_Button")
 		(at 260.35 138.43 0)
@@
 	(symbol
 		(lib_id "power:+3V3")
-		(at 154.94 119.38 0)
+		(at 152.4 119.38 0)
 		(mirror y)
 		(unit 1)
@@
 		(dnp no)
 		(property "Reference" "#PWR032"
-			(at 154.94 123.19 0)
+			(at 152.4 123.19 0)
 			(effects
 				(font
@@
 		)
 		(property "Value" "+3V3"
-			(at 154.94 114.3 0)
+			(at 152.4 114.3 0)
 			(effects
 				(font
@@
 		)
 		(property "Footprint" ""
-			(at 154.94 119.38 0)
+			(at 152.4 119.38 0)
 			(effects
 				(font
@@
 		)
 		(property "Datasheet" ""
-			(at 154.94 119.38 0)
+			(at 152.4 119.38 0)
 			(effects
 				(font
@@
 		)
 		(property "Description" "Power symbol creates a global label with name \"+3V3\""
-			(at 154.94 119.38 0)
+			(at 152.4 119.38 0)
 			(effects
 				(font
@@
 	)
 	(symbol
-		(lib_id "Jumper:Jumper_2_Bridged")
-		(at 162.56 127 0)
-		(unit 1)
-		(exclude_from_sim no)
-		(in_bom yes)
-		(on_board yes)
-		(dnp no)
-		(property "Reference" "JP2"
-			(at 162.306 128.778 0)
-			(effects
-				(font
-					(size 1.27 1.27)
-				)
-			)
-		)
-		(property "Value" "Jumper_2_Bridged"
-			(at 168.91 130.81 0)
-			(effects
-				(font
-					(size 1.27 1.27)
-				)
-			)
-		)
-		(property "Footprint" "Jumper:SolderJumper-2_P1.3mm_Bridged_RoundedPad1.0x1.5mm"
-			(at 162.56 127 0)
-			(effects
-				(font
-					(size 1.27 1.27)
-				)
-				(hide yes)
-			)
-		)
-		(property "Datasheet" "~"
-			(at 162.56 127 0)
-			(effects
-				(font
-					(size 1.27 1.27)
-				)
-				(hide yes)
-			)
-		)
-		(property "Description" "Jumper, 2-pole, closed/bridged"
-			(at 162.56 127 0)
-			(effects
-				(font
-					(size 1.27 1.27)
-				)
-				(hide yes)
-			)
-		)
-		(pin "1"
-		)
-		(pin "2"
-		)
-		(instances
-			(project ""
-				(path "/91d40f58-a363-48c7-98aa-eb2459062304"
-					(reference "JP2")
-					(unit 1)
-				)
-			)
-		)
-	)
-	(symbol
 		(lib_id "power:GND")
 		(at 243.84 52.07 270)
@@
 	)
 	(symbol
+		(lib_id "Jumper:SolderJumper_2_Bridged")
+		(at 161.29 119.38 0)
+		(unit 1)
+		(exclude_from_sim no)
+		(in_bom no)
+		(on_board yes)
+		(dnp no)
+		(property "Reference" "JP1"
+			(at 160.782 114.554 0)
+			(effects
+				(font
+					(size 1.27 1.27)
+				)
+			)
+		)
+		(property "Value" "SolderJumper_2_Bridged"
+			(at 169.418 116.84 0)
+			(effects
+				(font
+					(size 1.27 1.27)
+				)
+			)
+		)
+		(property "Footprint" "Jumper:SolderJumper-2_P1.3mm_Bridged_RoundedPad1.0x1.5mm"
+			(at 161.29 119.38 0)
+			(effects
+				(font
+					(size 1.27 1.27)
+				)
+				(hide yes)
+			)
+		)
+		(property "Datasheet" "~"
+			(at 161.29 119.38 0)
+			(effects
+				(font
+					(size 1.27 1.27)
+				)
+				(hide yes)
+			)
+		)
+		(property "Description" "Solder Jumper, 2-pole, closed/bridged"
+			(at 161.29 119.38 0)
+			(effects
+				(font
+					(size 1.27 1.27)
+				)
+				(hide yes)
+			)
+		)
+		(pin "2"
+		)
+		(pin "1"
+		)
+		(instances
+			(project ""
+				(path "/91d40f58-a363-48c7-98aa-eb2459062304"
+					(reference "JP1")
+					(unit 1)
+				)
+			)
+		)
+	)
+	(symbol
 		(lib_id "Device:R")
 		(at 227.33 110.49 0)
@@
 					(unit 1)
 				)
+			)
+		)
+	)
+	(symbol
+		(lib_id "Jumper:SolderJumper_2_Open")
+		(at 161.29 127 0)
+		(unit 1)
+		(exclude_from_sim no)
+		(in_bom no)
+		(on_board yes)
+		(dnp no)
+		(property "Reference" "JP2"
+			(at 161.29 129.794 0)
+			(effects
+				(font
+					(size 1.27 1.27)
+				)
+			)
+		)
+		(property "Value" "SolderJumper_2_Open"
+			(at 168.91 131.826 0)
+			(effects
+				(font
+					(size 1.27 1.27)
+				)
+			)
+		)
+		(property "Footprint" "Jumper:SolderJumper-2_P1.3mm_Open_RoundedPad1.0x1.5mm"
+			(at 161.29 127 0)
+			(effects
+				(font
+					(size 1.27 1.27)
+				)
+				(hide yes)
+			)
+		)
+		(property "Datasheet" "~"
+			(at 161.29 127 0)
+			(effects
+				(font
+					(size 1.27 1.27)
+				)
+				(hide yes)
+			)
+		)
+		(property "Description" "Solder Jumper, 2-pole, open"
+			(at 161.29 127 0)
+			(effects
+				(font
+					(size 1.27 1.27)
+				)
+				(hide yes)
+			)
+		)
+		(pin "2"
+		)
+		(pin "1"
+		)
+		(instances
+			(project ""
+				(path "/91d40f58-a363-48c7-98aa-eb2459062304"
+					(reference "JP2")
+					(unit 1)
+				)
